File: lume_hw/lume.sch (KiCad schematic (older format))
At the start: 39 parts, among them Q1 ALS-PT19-315C, SW1 BUTTON, SW2 BUTTON, SW3 BUTTON, SW4 BUTTON

Commit message: 24 hyperminutes
Parts:
- B1: symbol BAT -> lume-rescue:BAT
- C1, C10, C11, C13, C14, C2, C3, C4, C5, C6, C7, C8, C9: symbol C -> lume-rescue:C
- D1: symbol D_Shottky -> lume-rescue:D_Shottky
- DA1: symbol NCP583SQ -> lume-rescue:NCP583SQ
- DA2: symbol MCP1700 -> lume-rescue:MCP1700
- DA3: symbol MC74VHC1 -> lume-rescue:MC74VHC1
- DD1: symbol STM32F072CxTx -> lume-rescue:STM32F072CxTx
- HOLE1, HOLE2, HOLE3, HOLE4: symbol HOLE_METALLED -> lume-rescue:HOLE_METALLED
- Logo1: symbol Logo -> lume-rescue:Logo
- Q1: symbol Phototransistor -> lume-rescue:Phototransistor
- R2, R3: symbol R -> lume-rescue:R
- SW1, SW2, SW3, SW4: symbol BUTTON -> lume-rescue:BUTTON
- TP1, TP2: symbol TESTPOINT -> lume-rescue:TESTPOINT
- XL1: symbol USB_MINI_B -> lume-rescue:USB_MINI_B
- XL2: symbol CONN_6 -> lume-rescue:CONN_6
- XL3: symbol CONN_NOKIA_LCD -> lume-rescue:CONN_NOKIA_LCD
- XL4: symbol CONN_3 -> lume-rescue:CONN_3
- XL8: symbol CONN_2 -> lume-rescue:CONN_2
- XTAL1: symbol CRYSTAL_H -> lume-rescue:CRYSTAL_H
Connections:
- wire segments 124 -> 151
